Commit message: added diff drive plugin for gazebo simulation

File: scrubber_description/urdf/robot_base.xacro (robot description, xacro)
@@ -26,6 +26,146 @@
         rpy="0 0 0" />
       <mass
-        value="30" />
+        value="0.3" />
       <inertia
+        ixx="1"
+        ixy="0"
+        ixz="0"
+        iyy="1"
+        iyz="0"
+        izz="1" />
+    </inertial>
+    <visual>
+      <origin
+        xyz="0 0 0"
+        rpy="0 0 0" />
+      <geometry>
+        <mesh
+          filename="package://scrubber_description/meshes/chassis.stl"/>
+      </geometry>
+      <material
+        name="">
+        <color
+          rgba="0.79216 0.81961 0.92549 1" />
+      </material>
+    </visual>
+    <collision>
+      <origin
+        xyz="0 0 0"
+        rpy="0 0 0" />
+      <geometry>
+        <mesh
+          filename="package://scrubber_description/meshes/chassis.stl" />
+      </geometry>
+    </collision>
+  </link>
+   <joint
+    name="JLEFT"
+    type="continuous">
+    <origin
+      xyz="0 0.175 0"
+      rpy="0 0 0" />
+    <parent
+      link="chassis" />
+    <child
+      link="LEFTWHEEL" />
+    <axis
+      xyz="0 1 0" />
+  </joint>
+  <link name="LEFTWHEEL">
+    <visual>
+      <geometry>
+        <cylinder length="0.05" radius="0.1"/>
+      </geometry>
+      <material name="black">
+        <color rgba="0 0 0 1"/>
+      </material>
+      <origin
+      xyz="0 0 0"
+      rpy="1.507 0 0" />
+    </visual>
+    <collision>
+    <origin
+      xyz="0 0 0"
+      rpy="1.507 0 0" />
+      <geometry>
+        <cylinder length="0.05" radius="0.1"/>
+      </geometry>
+    </collision>
+    <inertial>
+    <origin
+      xyz="0 0 0"
+      rpy="1.507 0 0" />
+      <mass value="0.3"/>
+      <inertia ixx="1" ixy="0.0" ixz="0.0" iyy="1" iyz="0.0" izz="1"/>
+    </inertial>
+  </link>
+  <joint
+    name="JRIGHT"
+    type="continuous">
+    <origin
+      xyz="0 -0.175 0"
+      rpy="0 0 0" />
+    <parent
+      link="chassis" />
+    <child
+      link="RIGHTWHEEL" />
+    <axis
+      xyz="0 1 0" />
+  </joint>
+  <link name="RIGHTWHEEL">
+    <visual>
+      <geometry>
+        <cylinder length="0.05" radius="0.1"/>
+      </geometry>
+      <material name="black">
+        <color rgba="0 0 0 1"/>
+      </material>
+      <origin
+      xyz="0 0 0"
+      rpy="1.507 0 0" />
+    </visual>
+    <collision>
+    <origin
+      xyz="0 0 0"
+      rpy="1.507 0 0" />
+      <geometry>
+        <cylinder length="0.05" radius="0.1"/>
+      </geometry>
+    </collision>
+    <inertial>
+    <origin
+      xyz="0 0 0"
+      rpy="1.507 0 0" />
+      <mass value="0.3"/>
+      <inertia ixx="1" ixy="0.0" ixz="0.0" iyy="1" iyz="0.0" izz="1" />
+    </inertial>
+  </link>
+  <joint
+    name="brush_joint"
+    type="fixed">
+    <origin
+      xyz="0.3 0.0 -0.09"
+      rpy="0 0 0 " />
+    <parent
+      link="chassis" />
+    <child
+      link="brush" />
+  </joint>
+     <link
+    name="brush">
+    <inertial>
+      <origin
+        xyz="0 0 0"
+        rpy="0 0 0" />
+      <mass
+        value="0.5" />
+        <inertia
+        ixx="1"
+        ixy="0"
+        ixz="0"
+        iyy="1"
+        iyz="0"
+        izz="1" />
+      <!--inertia
         ixx="0.28974"
         ixy="-0.003469"
@@ -33,13 +173,13 @@
         iyy="0.71812"
         iyz="-0.0010571"
-        izz="0.69853" />
-    </inertial>
-    <visual>
-      <origin
-        xyz="0 0 0"
-        rpy="0 0 0" />
-      <geometry>
-        <mesh
-          filename="package://scrubber_description/meshes/chassis.stl"/>
+        izz="0.69853" /-->
+    </inertial>
+    <visual>
+      <origin
+        xyz="0 0 0"
+        rpy="0 0 0" />
+      <geometry>
+        <mesh
+          filename="package://scrubber_description/meshes/brush.stl"/>
       </geometry>
       <material
@@ -55,140 +195,13 @@
       <geometry>
         <mesh
-          filename="package://scrubber_description/meshes/chassis.stl" />
-      </geometry>
-    </collision>
-  </link>
-   <joint
-    name="JLEFT"
-    type="continuous">
-    <origin
-      xyz="0 0.175 0"
-      rpy="0 0 0" />
-    <parent
-      link="chassis" />
-    <child
-      link="LEFTWHEEL" />
-    <axis
-      xyz="0 1 0" />
-  </joint>
-  <link name="LEFTWHEEL">
-    <visual>
-      <geometry>
-        <cylinder length="0.05" radius="0.1"/>
-      </geometry>
-      <material name="black">
-        <color rgba="0 0 0 1"/>
-      </material>
-      <origin
-      xyz="0 0 0"
-      rpy="1.507 0 0" />
-    </visual>
-    <collision>
-      <geometry>
-        <cylinder length="0.05" radius="0.1"/>
-      </geometry>
-    </collision>
-    <inertial>
-    <origin
-      xyz="0 0 0"
-      rpy="1.507 0 0" />
-      <mass value="10"/>
-      <inertia ixx="0.4" ixy="0.0" ixz="0.0" iyy="0.4" iyz="0.0" izz="0.2"/>
-    </inertial>
+          filename="package://scrubber_description/meshes/brush.stl" />
+      </geometry>
+    </collision>
   </link>
   <joint
-    name="JRIGHT"
-    type="continuous">
-    <origin
-      xyz="0 -0.175 0"
-      rpy="0 0 0" />
-    <parent
-      link="chassis" />
-    <child
-      link="RIGHTWHEEL" />
-    <axis
-      xyz="0 1 0" />
-  </joint>
-  <link name="RIGHTWHEEL">
-    <visual>
-      <geometry>
-        <cylinder length="0.05" radius="0.1"/>
-      </geometry>
-      <material name="black">
-        <color rgba="0 0 0 1"/>
-      </material>
-      <origin
-      xyz="0 0 0"
-      rpy="1.507 0 0" />
-    </visual>
-    <collision>
-      <geometry>
-        <cylinder length="0.05" radius="0.1"/>
-      </geometry>
-    </collision>
-    <inertial>
-    <origin
-      xyz="0 0 0"
-      rpy="1.507 0 0" />
-      <mass value="10"/>
-      <inertia ixx="0.4" ixy="0.0" ixz="0.0" iyy="0.4" iyz="0.0" izz="0.2"/>
-    </inertial>
-  </link>
-  <joint
-    name="brush_joint"
-    type="fixed">
-    <origin
-      xyz="0.3 0.0 -0.05"
-      rpy="0 0 0 " />
-    <parent
-      link="chassis" />
-    <child
-      link="brush" />
-  </joint>
-     <link
-    name="brush">
-    <inertial>
-      <origin
-        xyz="0 0 0"
-        rpy="0 0 0" />
-      <mass
-        value="2" />
-      <inertia
-        ixx="0.28974"
-        ixy="-0.003469"
-        ixz="0.037331"
-        iyy="0.71812"
-        iyz="-0.0010571"
-        izz="0.69853" />
-    </inertial>
-    <visual>
-      <origin
-        xyz="0 0 0"
-        rpy="0 0 0" />
-      <geometry>
-        <mesh
-          filename="package://scrubber_description/meshes/brush.stl"/>
-      </geometry>
-      <material
-        name="">
-        <color
-          rgba="0.79216 0.81961 0.92549 1" />
-      </material>
-    </visual>
-    <collision>
-      <origin
-        xyz="0 0 0"
-        rpy="0 0 0" />
-      <geometry>
-        <mesh
-          filename="package://scrubber_description/meshes/brush.stl" />
-      </geometry>
-    </collision>
-  </link>
-    <joint
     name="lidar_joint"
     type="fixed">
     <origin
-      xyz="0.35 0.0 0.225"
+      xyz="0.55 0.0 0.225"
       rpy="0 0 0 " />
     <parent
@@ -219,24 +232,24 @@
   </actuator>
 </transmission>
-<transmission name="back_left_trans">
-  <type>transmission_interface/SimpleTransmission</type>
-  <joint name="JBACKLEFT">
-    <hardwareInterface>hardware_interface/VelocityJointInterface</hardwareInterface>
-  </joint>
-  <actuator name="Back_Left_Motor">
-    <hardwareInterface>hardware_interface/VelocityJointInterface</hardwareInterface>
-    <mechanicalReduction>1</mechanicalReduction>
-  </actuator>
-</transmission>
-<transmission name="back_right_trans">
-  <type>transmission_interface/SimpleTransmission</type>
-  <joint name="JBACKRIGHT">
-    <hardwareInterface>hardware_interface/VelocityJointInterface</hardwareInterface>
-  </joint>
-  <actuator name="Back_Right_Motor">
-    <hardwareInterface>hardware_interface/VelocityJointInterface</hardwareInterface>
-    <mechanicalReduction>1</mechanicalReduction>
-  </actuator>
-</transmission>
 -->
+<transmission name="left_trans">
+  <type>transmission_interface/SimpleTransmission</type>
+  <joint name="JLEFT">
+    <hardwareInterface>hardware_interface/EffortJointInterface</hardwareInterface>
+  </joint>
+  <actuator name="Left_Motor">
+    <hardwareInterface>hardware_interface/EffortJointInterface</hardwareInterface>
+    <mechanicalReduction>1</mechanicalReduction>
+  </actuator>
+</transmission>
+<transmission name="right_trans">
+  <type>transmission_interface/SimpleTransmission</type>
+  <joint name="JRIGHT">
+    <hardwareInterface>hardware_interface/EffortJointInterface</hardwareInterface>
+  </joint>
+  <actuator name="Right_Motor">
+    <hardwareInterface>hardware_interface/EffortJointInterface</hardwareInterface>
+    <mechanicalReduction>1</mechanicalReduction>
+  </actuator>
+</transmission>
 </robot>
